File: electrical/electrical_schematic/electrical_schematic.kicad_sch (KiCad schematic)
At the start: 3 parts, among them J1 Raspberry_Pi_2_3, U1 BME280, U2 RPR-0521RS

Commit message: Finished most of Tasks.py, Remade main
Parts:
- added U3: ~, symbol Display_Waveshare:Waveshare-9904
Connections:
- net at J1.1 (3V3), J1.17 (3V3), U1.6 (VDDIO)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: now also U3.1 (3.3V)
- net at J1.14 (GND), J1.20 (GND), J1.25 (GND)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: now also U3.14 (GND), U3.20 (GND), U3.25 (GND), U3.9 (GND)
- net at J1.19 (MOSI0/GPIO10): now also U3.19 (P_MOSI)
- net at J1.2 (5V), J1.4 (5V): now also U3.17 (3.3V), U3.2 (5V), U3.4 (5V)
- net at J1.21 (MISO0/GPIO9): now also U3.21 (P_MISO)
- net at J1.24 (~{CE0}/GPIO8): now also U3.24 (P_CE0)
- net at J1.26 (~{CE1}/GPIO7): now also U3.26 (P_CE1)
